File: hw/sch_pcb/ADSBAFE01.kicad_pcb (KiCad board)
At the start: 2 copper layers, 50.3 x 50.3 mm, 60 parts, among them J1 HEADER_2x12_PARALLEL, J2 HEADER_2x03_PARALLEL, J3 MCX 6GHz 50R, M1 RFShield_TwoPieces, M2 HOLE, M3 HOLE, M4 HOLE, M5 HOLE, SW1 SN74LVC1G3157, SW2 SN74LVC1G3157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

Commit message: Layout improvements.
Routing:
- net +3V3: track 116.5 -> 118.5 mm
Changed lines of the file:
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@@
+	)
+	(segment
+		(start 140.7414 108.9586)
+		(end 139.3 110.4)
+		(width 0.3)
+		(layer "F.Cu")
+		(net 1)
 	)
 	(segment
@@
 	)
 	(segment
-		(start 139.3 104.7)
-		(end 139.3 110.4)
+		(start 162.2 114.2)
+		(end 156.8 114.2)
 		(width 0.3)
 		(layer "F.Cu")
@@
 	)
 	(segment
-		(start 162.2 114.2)
-		(end 156.8 114.2)
+		(start 138.9 117.3)
+		(end 137.1446 115.5446)
 		(width 0.3)
 		(layer "F.Cu")
@@
 	)
 	(segment
+		(start 137.1446 115.5446)
+		(end 134.0554 115.5446)
+		(width 0.3)
+		(layer "F.Cu")
+		(net 1)
+	)
+	(segment
 		(start 137.1 115.5)
 		(end 138.9 117.3)
@@
 	)
 	(segment
-		(start 138.9 117.3)
-		(end 133.9 117.3)
+		(start 139.3 104.7)
+		(end 140.7414 106.1414)
 		(width 0.3)
 		(layer "F.Cu")
+		(net 1)
+	)
+	(segment
+		(start 134.0554 115.5446)
+		(end 133.9 115.7)
+		(width 0.3)
+		(layer "F.Cu")
+		(net 1)
+	)
+	(segment
+		(start 140.7414 106.1414)
+		(end 140.7414 108.9586)
+		(width 0.3)
+		(layer "F.Cu")

Commit message: Move footprints to standard MLAB libraries.
Parts:
- U1: footprint ADSB_project_footprints:VSSOP-8_3x3mm_P0.65mm_small -> Package_SO:VSSOP-8_3x3mm_P0.65mm
- X1: footprint ADSB_project_footprints:Filter_SAW-6_3.8x3.8mm -> MLAB_SAW:Filter_SAW-6_3.8x3.8mm
Changed lines of the file:
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@@
 		)
 	)
-	(footprint "ADSB_project_footprints:VSSOP-8_3x3mm_P0.65mm_small"
+	(footprint "Package_SO:VSSOP-8_3x3mm_P0.65mm"
 		(layer "B.Cu")
 		(at 148.1 111.5 180)
@@
 		(tags "VSSOP SO JEDEC-MO-187-AA Texas_DGK0008A")
 		(property "Reference" "U1"
-			(at 0 -2.4 0)
-			(unlocked yes)
+			(at 0 2.45 0)
 			(layer "B.SilkS")
 			(effects
@@
 			)
 		)
-		(property "Standard Cost" "0.84"
-			(at 0 0 0)
-			(unlocked yes)
-			(layer "B.Fab")
-			(hide yes)
-			(effects
-				(font
-					(size 1 1)
-					(thickness 0.15)
-				)
-				(justify mirror)
-			)
-		)
-		(property "Note" ""
-			(at 0 0 0)
-			(unlocked yes)
-			(layer "B.Fab")
-			(hide yes)
-			(effects
-				(font
-					(size 1 1)
-					(thickness 0.15)
-				)
-				(justify mirror)
-			)
-		)
-		(property "OEM PN" "TLV3542IDGKR"
-			(at 0 0 0)
-			(unlocked yes)
-			(layer "B.Fab")
-			(hide yes)
-			(effects
-				(font
-					(size 1 1)
-					(thickness 0.15)
-				)
-				(justify mirror)
-			)
-		)
 		(property "MPN" "TLV3542IDGKR"
-			(at 0 0 0)
+			(at 0 0 180)
 			(unlocked yes)
 			(layer "B.Fab")
@@
 			)
 		)
-		(property "REV" ""
-			(at 0 0 0)
+		(property "UST_ID" ""
+			(at 0 0 180)
 			(unlocked yes)
 			(layer "B.Fab")
@@
 		)
 		(pad "1" smd roundrect
-			(at -2.2 0.975 180)
-			(size 1.6 0.45)
+			(at -2.1125 0.975 180)
+			(size 1.625 0.5)
 			(layers "B.Cu" "B.Mask" "B.Paste")
 			(roundrect_rratio 0.25)
@@
 		)
 		(pad "2" smd roundrect
-			(at -2.2 0.325 180)
-			(size 1.6 0.45)
+			(at -2.1125 0.325 180)
+			(size 1.625 0.5)
 			(layers "B.Cu" "B.Mask" "B.Paste")
 			(roundrect_rratio 0.25)
@@
 		)
 		(pad "3" smd roundrect
-			(at -2.2 -0.325 180)
-			(size 1.6 0.45)
+			(at -2.1125 -0.325 180)
+			(size 1.625 0.5)
 			(layers "B.Cu" "B.Mask" "B.Paste")
 			(roundrect_rratio 0.25)
@@
 		)
 		(pad "4" smd roundrect
-			(at -2.2 -0.975 180)
-			(size 1.6 0.45)
+			(at -2.1125 -0.975 180)
+			(size 1.625 0.5)
 			(layers "B.Cu" "B.Mask" "B.Paste")
 			(roundrect_rratio 0.25)
@@
 		)
 		(pad "5" smd roundrect
-			(at 2.2 -0.975 180)
-			(size 1.6 0.45)
+			(at 2.1125 -0.975 180)
+			(size 1.625 0.5)
 			(layers "B.Cu" "B.Mask" "B.Paste")
 			(roundrect_rratio 0.25)
@@
 		)
 		(pad "6" smd roundrect
-			(at 2.2 -0.325 180)
-			(size 1.6 0.45)
+			(at 2.1125 -0.325 180)
+			(size 1.625 0.5)
 			(layers "B.Cu" "B.Mask" "B.Paste")
 			(roundrect_rratio 0.25)
@@
 		)
 		(pad "7" smd roundrect
-			(at 2.2 0.325 180)
-			(size 1.6 0.45)
+			(at 2.1125 0.325 180)
+			(size 1.625 0.5)
 			(layers "B.Cu" "B.Mask" "B.Paste")
 			(roundrect_rratio 0.25)
@@
 		)
 		(pad "8" smd roundrect
-			(at 2.2 0.975 180)
-			(size 1.6 0.45)
+			(at 2.1125 0.975 180)
+			(size 1.625 0.5)
 			(layers "B.Cu" "B.Mask" "B.Paste")
 			(roundrect_rratio 0.25)
@@
 		)
 	)
-	(footprint "ADSB_project_footprints:Filter_SAW-6_3.8x3.8mm"
+	(footprint "MLAB_SAW:Filter_SAW-6_3.8x3.8mm"
 		(layer "B.Cu")
 		(at 151.84 99.325 -90)
@@
 		(tags "SAW filter 6-pin")
 		(property "Reference" "X1"
-			(at -0.425 3.14 90)
-			(unlocked yes)
+			(at 0.01 -3.22 270)
 			(layer "B.SilkS")
+			(hide yes)
 			(effects
 				(font
@@
 		)
 		(property "Value" "SF2321D"
-			(at 0.01 3.59 90)
+			(at 0.01 3.59 270)
 			(layer "B.Fab")
 			(effects
@@
 		)
 		(property "Standard Cost" "1.10"
-			(at 0 0 0)
+			(at 0 0 180)
 			(layer "B.Fab")
 			(hide yes)
@@
 			)
 		)
-		(property "REV" ""
-			(at 0 0 90)
+		(property "UST_ID" ""
+			(at 0 0 270)
 			(unlocked yes)
 			(layer "B.Fab")
@@
 		)
 		(fp_text user "${REFERENCE}"
-			(at -0.02 -0.01 90)
+			(at -0.02 -0.01 270)
 			(layer "B.Fab")
 			(effects
@@
 		)
 		(embedded_fonts no)
-		(model "${KIPRJMOD}/3d_models/SF2321D--3DModel-STEP-672324.STEP"
+		(model "${KICAD_LIBS_DIR}/lib_3d/Custom_Filter/Filter_SAW-6_3.8x3.8mm.stp"
 			(offset
-				(xyz 0 0 0)
+				(xyz 0 1.15 0)
 			)
 			(scale
@@
 			)
 			(rotate
-				(xyz -0 -0 -0)
+				(xyz 0 0 90)
 			)
 		)
